Commit message: 完成导航实现,部分bug需要修复

File: src/sim_dog/go2_description/urdf/go2_description_ign.urdf (robot description, URDF)
Before this commit: robot go2_description, 42 links, 41 joints
Links:
- added link laser_up
Joints:
- added joint laser_joint: type fixed, parent base, child laser_up, origin xyz=0.0 0.0 0.2 rpy=0.0 0.0 0.0, axis 0.0 0.0 0.0, limit lower=0.0 upper=0.0 effort=0.0 velocity=0.0

Commit message: 修改部分参数

File: src/sim_dog/go2_description/urdf/go2_description_ign.urdf (robot description, URDF)
Before this commit: robot go2_description, 43 links, 42 joints
Joints:
- joint laser_joint: origin xyz=0.0 0.0 0.2 rpy=0.0 0.0 0.0 -> xyz=0.0 0.0 0.1 rpy=0.0 0.0 0.0

Commit message: imu传感器添加

File: src/sim_dog/go2_description/urdf/go2_description_ign.urdf (robot description, URDF)
Before this commit: robot go2_description, 43 links, 42 joints
Links:
- link imu: mass 0 -> None
